Commit message: Update cart.xacro

File: cart_description/urdf/cart.xacro (robot description, xacro)
@@ -88,5 +88,5 @@
   <parent link="base_link"/>
   <child link="wheel__1_1"/>
-  <axis xyz="0.0 -1.0 -0.0"/>
+  <axis xyz="0.0 1.0 0.0"/>
 </joint>
 <joint name="Rev2" type="continuous">
@@ -94,5 +94,5 @@
   <parent link="base_link"/>
   <child link="wheel_2_1"/>
-  <axis xyz="-0.0 1.0 0.0"/>
+  <axis xyz="0.0 1.0 0.0"/>
 </joint>
 <joint name="Rev3" type="continuous">
@@ -100,5 +100,5 @@
   <parent link="base_link"/>
   <child link="revert_1_1"/>
-  <axis xyz="0.0 -0.0 1.0"/>
+  <axis xyz="0.0 0.0 1.0"/>
 </joint>
 </robot>
